File: Hardware/Rele-wifi De Caro.kicad_pcb (KiCad board)
At the start: 2 copper layers, 11 parts, among them J1 Screw_Terminal_01x03, J2 Screw_Terminal_01x03, J3 Screw_Terminal_01x03, J4 Screw_Terminal_01x03, J5 Screw_Terminal_01x02, Q2 PC817-B, Q4 PC817-B, Q5 PC817-B, Q7 PC817-B, U2 ESP32-CAM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

Commit message: Avance de esquematico
Parts:
- added K1: Relay_SPDT, Relay:RELAY_PR13-5V-450-1C, F.Cu at (107.0, 60.3)
- added K2: Relay_SPDT, Relay:RELAY_PR13-5V-450-1C, F.Cu at (107.0, 77.4)
- added K3: Relay_SPDT, Relay:RELAY_PR13-5V-450-1C, F.Cu at (107.0, 94.4)
- added K5: Relay_SPDT, Relay:RELAY_PR13-5V-450-1C, F.Cu at (107.0, 111.5)
Connections:
- U2 pad P$1: Net-(U1-OUT) -> Net-(U2-5V)
- U3 pad 1: unconnected-(U3-VI-Pad1) -> Net-(SW1A-B)
- U3 pad 2: unconnected-(U3-GND-Pad2) -> GND
- U3 pad 3: unconnected-(U3-VO-Pad3) -> Net-(U2-5V)

Commit message: Avance pcb
Parts:
- removed K5: Relay_SPDT, Relay:RELAY_PR13-5V-450-1C
- removed U3: LM7805_TO220, Package_TO_SOT_THT:TO-220-3_Vertical
- added 10K1: R, Resistor_SMD:R_0805_2012Metric_Pad1.20x1.40mm_HandSolder, F.Cu at (173.0, 65.5)
- added 10K2: R, Resistor_SMD:R_0805_2012Metric_Pad1.20x1.40mm_HandSolder, F.Cu at (173.0, 47.5)
- added 10K3: R, Resistor_SMD:R_0805_2012Metric_Pad1.20x1.40mm_HandSolder, F.Cu at (43.9, 150.7)
- added 10K4: R, Resistor_SMD:R_0805_2012Metric_Pad1.20x1.40mm_HandSolder, F.Cu at (43.9, 153.7)
- added C5: 0.1uF, Capacitor_SMD:C_0805_2012Metric, F.Cu at (65.5, 162.5)
- added C6: 0.1uF, Capacitor_SMD:C_0805_2012Metric, F.Cu at (65.5, 165.5)
- added D1: LED, LED_SMD:LED_0805_2012Metric, F.Cu at (39.4, 144.9)
- added D2: LED, LED_SMD:LED_0805_2012Metric, F.Cu at (161.5, 56.0)
- added D3: D, Diode_SMD:D_0805_2012Metric, F.Cu at (173.0, 56.5)
- added D4: D, Diode_SMD:D_0805_2012Metric, F.Cu at (173.1, 74.5)
- added D5: LED, LED_SMD:LED_0805_2012Metric, F.Cu at (39.4, 157.0)
- added D6: D, Diode_SMD:D_0805_2012Metric, F.Cu at (39.4, 160.1)
- added D7: LED, LED_SMD:LED_0805_2012Metric, F.Cu at (39.4, 163.1)
- added D8: D, Diode_SMD:D_0805_2012Metric, F.Cu at (39.4, 166.2)
- added IC1: MC7805CD2TG, 7805 d2pak:MC7805CD2TG, F.Cu at (57.5, 152.4)
- added K4: PR13-5V-450-1C, relay:RELAY_PR13-5V-450-1C, F.Cu at (186.0, 106.0)
- added Q1: PC817-B, optoacoplador:SOT254P1025X400-4N, F.Cu at (166.7, 70.0)
- added Q3: BC547, bc547 smd:SOT95P230X110-3N, F.Cu at (173.0, 52.0)
- added Q6: BC547, bc547 smd:SOT95P230X110-3N, F.Cu at (49.4, 154.5)
- added Q8: BC547, bc547 smd:SOT95P230X110-3N, F.Cu at (49.4, 158.9)
- added R1: 220, Resistor_SMD:R_0805_2012Metric_Pad1.20x1.40mm_HandSolder, F.Cu at (43.9, 156.6)
- added R2: 220, Resistor_SMD:R_0805_2012Metric_Pad1.20x1.40mm_HandSolder, F.Cu at (161.5, 51.0)
- added R3: 220, Resistor_SMD:R_0805_2012Metric_Pad1.20x1.40mm_HandSolder, F.Cu at (43.9, 162.5)
- added R4: 220, Resistor_SMD:R_0805_2012Metric_Pad1.20x1.40mm_HandSolder, F.Cu at (43.9, 165.5)
- K1, K2, K3: value Relay_SPDT -> PR13-5V-450-1C; footprint Relay:RELAY_PR13-5V-450-1C -> relay:RELAY_PR13-5V-450-1C
- Q2, Q5, Q7: footprint Optocoplador:SOT254P1025X400-4N -> optoacoplador:SOT254P1025X400-4N
- Q4: value PC817-B -> BC547; footprint Optocoplador:SOT254P1025X400-4N -> bc547 smd:SOT95P230X110-3N
- U2: footprint ESP32 cam:ESP32-CAM -> esp cam:ESP32-CAM
- moved Q7 145.3 mm to (24.5, 113.5)
- moved Q5 145.1 mm to (24.5, 105.5)
- moved J5 124.8 mm to (55.0, 165.5)
- moved K1 79.4 mm to (186.0, 52.0)
- moved K2 79.3 mm to (186.0, 70.0)
- moved K3 79.2 mm to (186.0, 88.0)
- moved J2 64.5 mm to (202.0, 46.9), turned to -90 degrees
- moved J3 54.3 mm to (202.0, 82.8), turned to -90 degrees
- moved J1 54.3 mm to (202.0, 64.8), turned to -90 degrees
- moved J4 53.5 mm to (202.0, 100.8), turned to -90 degrees
- moved U2 21.3 mm to (145.1, 68.8), turned to 180 degrees
- moved Q2 20.7 mm to (167.0, 52.0), turned to 90 degrees
- moved Q4 10.5 mm to (173.0, 70.0), turned to 180 degrees
Connections:
- J1 pad 1: 12 -> Net-(J1-Pin_1)
- J1 pad 2: 11 -> Net-(J1-Pin_2)
- J1 pad 3: 14 -> Net-(J1-Pin_3)
- J2 pad 1: 12 -> Net-(J2-Pin_1)
- J2 pad 2: 11 -> Net-(J2-Pin_2)
- J2 pad 3: 14 -> Net-(J2-Pin_3)
- J3 pad 1: 12 -> Net-(J3-Pin_1)
- J3 pad 2: 11 -> Net-(J3-Pin_2)
- J3 pad 3: 14 -> Net-(J3-Pin_3)
- J4 pad 1: 12 -> Net-(J4-Pin_1)
- J4 pad 2: 11 -> Net-(J4-Pin_2)
- J4 pad 3: 14 -> Net-(J4-Pin_3)
- K1 pad COM: (no net) -> Net-(J2-Pin_2)
- K1 pad NC: (no net) -> Net-(J2-Pin_1)
- K1 pad NO: (no net) -> Net-(J2-Pin_3)
- K2 pad A2: Net-(D6-A) (its old number) -> Net-(D4-A)
- K2 pad COM: (no net) -> Net-(J1-Pin_2)
- K2 pad NC: (no net) -> Net-(J1-Pin_1)
- K2 pad NO: (no net) -> Net-(J1-Pin_3)
- K3 pad COM: (no net) -> Net-(J3-Pin_2)
- K3 pad NC: (no net) -> Net-(J3-Pin_1)
- K3 pad NO: (no net) -> Net-(J3-Pin_3)
- Q4 pad 1: Net-(Q4-Pad1) -> Net-(D4-A)
- Q4 pad 2: GND -> Net-(Q4-B)
- Q4 pad 3: Net-(10K2-Pad2) (its old number) -> GND
- U2 pad P$9: unconnected-(U2-.GND-PadP$9) -> GND
